Commit message: fix(urdf): add missing position interfaces

File: src/mach_description/urdf/bfmc_car.urdf.xacro (robot description, xacro)
@@ -266,21 +266,12 @@
     <joint name="rear_left_wheel_joint">
       <command_interface name="velocity"/>
+      <state_interface name="position"/>
       <state_interface name="velocity"/>
     </joint>
     <joint name="rear_right_wheel_joint">
       <command_interface name="velocity"/>
+      <state_interface name="position"/>
       <state_interface name="velocity"/>
     </joint>
-<!--Added for testing-->
-<!--
-    <joint name="front_left_wheel_joint">
-      <state_interface name="velocity"/>
-      <state_interface name="position"/>
-    </joint>
-    <joint name="front_right_wheel_joint">
-      <state_interface name="velocity"/>
-      <state_interface name="position"/>
-    </joint>
--->
     <joint name="front_left_wheel_joint">
       <command_interface name="position"/>

Commit message: feat(sim): add ROS 2 Gazebo simulator
* Added Mach Simulator

* fix(sim): gazebo launching errors

* refactor(description): move urdf to mach_description

* fix(urdf): add missing position interfaces

* feat(sim): add rviz config

* refactor(sim): move simulation dependencies to mach_simulation

---------

Co-authored-by: Hiba Anwar <hiba2anwar@gmail.com>

File: src/mach_description/urdf/bfmc_car.urdf.xacro (robot description, xacro)
@@ -5,7 +5,7 @@
   <!--  -->
   <xacro:property name="PI" value="3.14159265359"/>
-  <!-- Chassis dimensions and mass -->
+  <!-- Chassis dimensions and mass 0.18 -->
   <xacro:property name="chassis_len"    value="0.30"/>
-  <xacro:property name="chassis_width"  value="0.18"/>
+  <xacro:property name="chassis_width"  value="0.12"/>
   <xacro:property name="chassis_height" value="0.05"/>
   <xacro:property name="chassis_mass"   value="1.5"/>
@@ -250,3 +250,95 @@
   <!-- Front Right Steering Link -->
   <xacro:front_steering prefix="front_right" y_pos="-${track_width/2}"/>
+  <ros2_control name="BFMCSystem" type="system">
+    <hardware>
+      <plugin>gazebo_ros2_control/GazeboSystem</plugin>
+    </hardware>
+    <!-- Steering joints -->
+    <joint name="front_left_steering_joint">
+      <command_interface name="position"/>
+      <state_interface name="position"/>
+    </joint>
+    <joint name="front_right_steering_joint">
+      <command_interface name="position"/>
+      <state_interface name="position"/>
+    </joint>
+    <!-- Rear wheels -->
+    <joint name="rear_left_wheel_joint">
+      <command_interface name="velocity"/>
+      <state_interface name="position"/>
+      <state_interface name="velocity"/>
+    </joint>
+    <joint name="rear_right_wheel_joint">
+      <command_interface name="velocity"/>
+      <state_interface name="position"/>
+      <state_interface name="velocity"/>
+    </joint>
+    <joint name="front_left_wheel_joint">
+      <command_interface name="position"/>
+      <state_interface name="position"/>
+    </joint>
+    <joint name="front_right_wheel_joint">
+      <command_interface name="position"/>
+      <state_interface name="position"/>
+    </joint>
+  </ros2_control>
+  <!-- LEFT CAMERA -->
+  <gazebo reference="camera_left">
+    <sensor type="camera" name="left_camera">
+      <update_rate>30</update_rate>
+      <camera>
+        <horizontal_fov>1.396</horizontal_fov>
+        <image>
+          <width>640</width>
+          <height>480</height>
+          <format>R8G8B8</format>
+        </image>
+        <clip>
+          <near>0.05</near>
+          <far>50</far>
+        </clip>
+      </camera>
+      <plugin name="gazebo_ros_camera_left" filename="libgazebo_ros_camera.so">
+        <ros>
+          <namespace>/camera</namespace>
+        </ros>
+        <camera_name>left</camera_name>
+        <image_topic_name>image_raw</image_topic_name>
+        <frame_name>camera_left_optical</frame_name>
+      </plugin>
+    </sensor>
+  </gazebo>
+  <!-- RIGHT CAMERA -->
+  <gazebo reference="camera_right">
+    <sensor type="camera" name="right_camera">
+      <update_rate>30</update_rate>
+      <camera>
+        <horizontal_fov>1.396</horizontal_fov>
+        <image>
+          <width>640</width>
+          <height>480</height>
+          <format>R8G8B8</format>
+        </image>
+        <clip>
+          <near>0.05</near>
+          <far>50</far>
+        </clip>
+      </camera>
+      <plugin name="gazebo_ros_camera_right" filename="libgazebo_ros_camera.so">
+        <ros>
+          <namespace>/camera</namespace>
+        </ros>
+        <camera_name>right</camera_name>
+        <image_topic_name>image_raw</image_topic_name>
+        <frame_name>camera_right_optical</frame_name>
+      </plugin>
+    </sensor>
+  </gazebo>
+  <gazebo>
+    <plugin name="gazebo_ros2_control" filename="libgazebo_ros2_control.so">
+      <robot_param>robot_description</robot_param>
+      <robot_param_node>robot_state_publisher</robot_param_node>
+      <parameters>$(find mach_simulator)/config/ros2_control.yaml</parameters>
+    </plugin>
+  </gazebo>
 </robot>

Commit message: feat(sim): add lane_detection node

File: src/mach_description/urdf/bfmc_car.urdf.xacro (robot description, xacro)
@@ -6,5 +6,5 @@
   <xacro:property name="PI" value="3.14159265359"/>
   <!-- Chassis dimensions and mass 0.18 -->
-  <xacro:property name="chassis_len"    value="0.30"/>
+  <xacro:property name="chassis_len"    value="0.36"/>
   <xacro:property name="chassis_width"  value="0.12"/>
   <xacro:property name="chassis_height" value="0.05"/>
@@ -112,7 +112,5 @@
       <parent link="base_link"/>
       <child link="camera_${prefix}"/>
-      <origin
-        xyz="${chassis_x_offset + chassis_len/2 - 0.01} ${y_offset} ${chassis_z_offset + chassis_height + 0.01}"
-        rpy="0 0 0"/>
+      <origin xyz="0.15 ${y_offset} 0.17" rpy="0 0 0"/>
     </joint>
     <!-- Optical frame (ROS camera convention) -->

Commit message: Project Status 2 (#12)
* feat(sim): add ROS 2 Gazebo simulator

* Added Mach Simulator

* fix(sim): gazebo launching errors

* refactor(description): move urdf to mach_description

* fix(urdf): add missing position interfaces

* feat(sim): add rviz config

* refactor(sim): move simulation dependencies to mach_simulation

---------

Co-authored-by: Hiba Anwar <hiba2anwar@gmail.com>

* feat(sim): fix ackermann control pipeline (#9)

* feat(sim): add ackermann to twist node

* fix(sim): ackermann steering mismatch

* refactor(sim): update twist to twist_stamped

* feat(camera): stereo camera bringup and calibration (#8)

* refactor(nucleo): rename package to mach_hardware

* feat(hardware): add stereo camera launch

* feat(camera): add camera calibration config

* feat(sim): add lane_detection node (#10)

- `mach_perception` python package with the lane detection node

* feat(control): PID lane following (#11)

* feat(control): add PID lane follower

* feat(control): integrate lane following with detection

* project status 2

---------

Co-authored-by: Abyaz34 <128247302+Abyaz34@users.noreply.github.com>

File: src/mach_description/urdf/bfmc_car.urdf.xacro (robot description, xacro)
@@ -5,7 +5,7 @@
   <!--  -->
   <xacro:property name="PI" value="3.14159265359"/>
-  <!-- Chassis dimensions and mass -->
-  <xacro:property name="chassis_len"    value="0.30"/>
-  <xacro:property name="chassis_width"  value="0.18"/>
+  <!-- Chassis dimensions and mass 0.18 -->
+  <xacro:property name="chassis_len"    value="0.36"/>
+  <xacro:property name="chassis_width"  value="0.12"/>
   <xacro:property name="chassis_height" value="0.05"/>
   <xacro:property name="chassis_mass"   value="1.5"/>
@@ -112,7 +112,5 @@
       <parent link="base_link"/>
       <child link="camera_${prefix}"/>
-      <origin
-        xyz="${chassis_x_offset + chassis_len/2 - 0.01} ${y_offset} ${chassis_z_offset + chassis_height + 0.01}"
-        rpy="0 0 0"/>
+      <origin xyz="0.15 ${y_offset} 0.17" rpy="0 0 0"/>
     </joint>
     <!-- Optical frame (ROS camera convention) -->
@@ -247,6 +245,100 @@
   </xacro:macro>
   <!-- Front Left Steering Link -->
-  <xacro:front_steering prefix="front_left"  y_pos="${track_width/2}"/>
+  <xacro:front_steering prefix="front_left" y_pos="${track_width/2}"/>
   <!-- Front Right Steering Link -->
   <xacro:front_steering prefix="front_right" y_pos="-${track_width/2}"/>
+  <ros2_control name="BFMCSystem" type="system">
+    <hardware>
+      <plugin>gazebo_ros2_control/GazeboSystem</plugin>
+    </hardware>
+    <!-- Steering joints -->
+    <joint name="front_left_steering_joint">
+      <command_interface name="position"/>
+      <state_interface name="position"/>
+    </joint>
+    <joint name="front_right_steering_joint">
+      <command_interface name="position"/>
+      <state_interface name="position"/>
+    </joint>
+    <!-- Rear wheels -->
+    <joint name="rear_left_wheel_joint">
+      <command_interface name="velocity"/>
+      <state_interface name="position"/>
+      <state_interface name="velocity"/>
+    </joint>
+    <joint name="rear_right_wheel_joint">
+      <command_interface name="velocity"/>
+      <state_interface name="position"/>
+      <state_interface name="velocity"/>
+    </joint>
+    <joint name="front_left_wheel_joint">
+      <!-- <command_interface name="position"/> -->
+      <state_interface name="velocity"/>
+      <state_interface name="position"/>
+    </joint>
+    <joint name="front_right_wheel_joint">
+      <!-- <command_interface name="position"/> -->
+      <state_interface name="velocity"/>
+      <state_interface name="position"/>
+    </joint>
+  </ros2_control>
+  <!-- LEFT CAMERA -->
+  <gazebo reference="camera_left">
+    <sensor type="camera" name="left_camera">
+      <update_rate>30</update_rate>
+      <camera>
+        <horizontal_fov>1.396</horizontal_fov>
+        <image>
+          <width>640</width>
+          <height>480</height>
+          <format>R8G8B8</format>
+        </image>
+        <clip>
+          <near>0.05</near>
+          <far>50</far>
+        </clip>
+      </camera>
+      <plugin name="gazebo_ros_camera_left" filename="libgazebo_ros_camera.so">
+        <ros>
+          <namespace>/camera</namespace>
+        </ros>
+        <camera_name>left</camera_name>
+        <image_topic_name>image_raw</image_topic_name>
+        <frame_name>camera_left_optical</frame_name>
+      </plugin>
+    </sensor>
+  </gazebo>
+  <!-- RIGHT CAMERA -->
+  <gazebo reference="camera_right">
+    <sensor type="camera" name="right_camera">
+      <update_rate>30</update_rate>
+      <camera>
+        <horizontal_fov>1.396</horizontal_fov>
+        <image>
+          <width>640</width>
+          <height>480</height>
+          <format>R8G8B8</format>
+        </image>
+        <clip>
+          <near>0.05</near>
+          <far>50</far>
+        </clip>
+      </camera>
+      <plugin name="gazebo_ros_camera_right" filename="libgazebo_ros_camera.so">
+        <ros>
+          <namespace>/camera</namespace>
+        </ros>
+        <camera_name>right</camera_name>
+        <image_topic_name>image_raw</image_topic_name>
+        <frame_name>camera_right_optical</frame_name>
+      </plugin>
+    </sensor>
+  </gazebo>
+  <gazebo>
+    <plugin name="gazebo_ros2_control" filename="libgazebo_ros2_control.so">
+      <robot_param>robot_description</robot_param>
+      <robot_param_node>robot_state_publisher</robot_param_node>
+      <parameters>$(find mach_simulator)/config/ros2_control.yaml</parameters>
+    </plugin>
+  </gazebo>
 </robot>
